File: V2.0.0/Dev Board/Dev Board.sch (KiCad schematic (older format))
At the start: 57 parts, among them J1 PICKIT4 Conn, J2 I2C Conn, J3 UART Conn, J4 SPI Conn, J5 CAN Conn, J6 PORT B, J7 Analog, U1 MCP2551-I-SN, U2 PIC18F25K80_ISS, U3 NCP1117-5.0_TO252, Y1 20MHz

Commit message: PGD and PGC Glitch Removed
Changed lines of the file:
@@
 Text Label 3600 3350 2    50   ~ 0
 ~MCLR
+Text Label 3600 2950 2    50   ~ 0
+RB6_PGC
 Text Label 3600 3050 2    50   ~ 0
-RB6_PGC
-Text Label 3600 2950 2    50   ~ 0
 RB7_PGD
 Wire Wire Line
